File: pcb/counter_reset_signal_conditioning.kicad_sch (KiCad schematic)
At the start: 3 parts

Commit message: added 2nd revision (PCB + PIO-based firmware)
Parts:
- added C?: 220nF, symbol Device:C
Connections:
- net GND: now also C?.2
- net Signal_3V3: now also C?.1
Changed lines of the file:
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@@
 (kicad_sch (version 20211123) (generator eeschema)
   (paper "A4")
+  (junction (at 93.98 110.49) (diameter 0) (color 0 0 0 0)
+  )
+  (junction (at 101.6 99.06) (diameter 0) (color 0 0 0 0)
+  )
   (junction (at 93.98 99.06) (diameter 0) (color 0 0 0 0)
-  )
-  (wire (pts (xy 93.98 104.14) (xy 93.98 109.22))
-    (stroke (width 0) (type default) (color 0 0 0 0))
   )
   (wire (pts (xy 68.58 99.06) (xy 73.66 99.06))
     (stroke (width 0) (type default) (color 0 0 0 0))
   )
-  (wire (pts (xy 93.98 99.06) (xy 99.06 99.06))
+  (wire (pts (xy 93.98 99.06) (xy 101.6 99.06))
     (stroke (width 0) (type default) (color 0 0 0 0))
   )
   (wire (pts (xy 93.98 86.36) (xy 93.98 88.9))
+    (stroke (width 0) (type default) (color 0 0 0 0))
+  )
+  (wire (pts (xy 101.6 99.06) (xy 101.6 101.6))
+    (stroke (width 0) (type default) (color 0 0 0 0))
+  )
+  (wire (pts (xy 93.98 110.49) (xy 93.98 111.76))
     (stroke (width 0) (type default) (color 0 0 0 0))
   )
@@
     (stroke (width 0) (type default) (color 0 0 0 0))
   )
+  (wire (pts (xy 101.6 99.06) (xy 104.14 99.06))
+    (stroke (width 0) (type default) (color 0 0 0 0))
+  )
   (wire (pts (xy 93.98 96.52) (xy 93.98 99.06))
     (stroke (width 0) (type default) (color 0 0 0 0))
   )
   (wire (pts (xy 68.58 81.28) (xy 68.58 86.36))
+    (stroke (width 0) (type default) (color 0 0 0 0))
+  )
+  (wire (pts (xy 93.98 110.49) (xy 101.6 110.49))
     (stroke (width 0) (type default) (color 0 0 0 0))
   )
@@
     (stroke (width 0) (type default) (color 0 0 0 0))
   )
-  (hierarchical_label "Signal_3V3" (shape output) (at 99.06 99.06 0)
+  (wire (pts (xy 101.6 109.22) (xy 101.6 110.49))
+    (stroke (width 0) (type default) (color 0 0 0 0))
+  )
+  (wire (pts (xy 93.98 104.14) (xy 93.98 110.49))
+    (stroke (width 0) (type default) (color 0 0 0 0))
+  )
+  (hierarchical_label "Signal_3V3" (shape output) (at 104.14 99.06 0)
     (effects (font (size 1.27 1.27)) (justify left))
   )
   (hierarchical_label "Signal_12V" (shape input) (at 63.5 81.28 180)
     (effects (font (size 1.27 1.27)) (justify right))
+  )
+  (symbol (lib_id "Device:C") (at 101.6 105.41 0) (unit 1)
+    (in_bom yes) (on_board yes) (fields_autoplaced)
+    (property "Reference" "C?" (id 0) (at 105.41 104.1399 0)
+      (effects (font (size 1.27 1.27)) (justify left))
+    )
+    (property "Value" "220nF" (id 1) (at 105.41 106.6799 0)
+      (effects (font (size 1.27 1.27)) (justify left))
+    )
+    (property "Footprint" "" (id 2) (at 102.5652 109.22 0)
+      (effects (font (size 1.27 1.27)) hide)
+    )
+    (property "Datasheet" "~" (id 3) (at 101.6 105.41 0)
+      (effects (font (size 1.27 1.27)) hide)
+    )
+    (pin "1")
+    (pin "2")
   )
   (symbol (lib_id "power:+3V3") (at 93.98 86.36 0) (unit 1)
@@
     (pin "2")
   )
-  (symbol (lib_id "power:GND") (at 93.98 109.22 0) (unit 1)
+  (symbol (lib_id "power:GND") (at 93.98 111.76 0) (unit 1)
     (in_bom yes) (on_board yes)
-    (property "Reference" "#PWR?" (id 0) (at 93.98 115.57 0)
+    (property "Reference" "#PWR?" (id 0) (at 93.98 118.11 0)
       (effects (font (size 1.27 1.27)) hide)
     )
-    (property "Value" "GND" (id 1) (at 93.98 114.3 0))
-    (property "Footprint" "" (id 2) (at 93.98 109.22 0)
+    (property "Value" "GND" (id 1) (at 93.98 116.84 0))
+    (property "Footprint" "" (id 2) (at 93.98 111.76 0)
       (effects (font (size 1.27 1.27)) hide)
     )
-    (property "Datasheet" "" (id 3) (at 93.98 109.22 0)
+    (property "Datasheet" "" (id 3) (at 93.98 111.76 0)
       (effects (font (size 1.27 1.27)) hide)
     )
