File: pcb/indoor_power_ctrl_signal_conditioning.kicad_sch (KiCad schematic)
At the start: 3 parts

Commit message: added 2nd revision (PCB + PIO-based firmware)
Parts:
- added C?: 220nF, symbol Device:C
- R?: value 600R -> 1k
Connections:
- net +3V3: now also R?.1; no longer U?.4 (R)
- net GND: now also U?.3 (R), C?.2; no longer R?.2
- net Signal_3V3: now also R?.2, U?.4 (R), C?.1; no longer R?.1, U?.3 (R)
Other:
- moved on the sheet: R?
Changed lines of the file:
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@@
 (kicad_sch (version 20211123) (generator eeschema)
   (paper "A4")
-  (junction (at 132.08 102.87) (diameter 0) (color 0 0 0 0)
+  (junction (at 132.08 97.79) (diameter 0) (color 0 0 0 0)
+  )
+  (junction (at 132.08 109.22) (diameter 0) (color 0 0 0 0)
+  )
+  (junction (at 139.7 97.79) (diameter 0) (color 0 0 0 0)
+  )
+  (wire (pts (xy 132.08 97.79) (xy 139.7 97.79))
+    (stroke (width 0) (type default) (color 0 0 0 0))
   )
   (wire (pts (xy 132.08 97.79) (xy 127 97.79))
     (stroke (width 0) (type default) (color 0 0 0 0))
   )
-  (wire (pts (xy 106.68 97.79) (xy 111.76 97.79))
+  (wire (pts (xy 132.08 102.87) (xy 132.08 109.22))
     (stroke (width 0) (type default) (color 0 0 0 0))
   )
-  (wire (pts (xy 132.08 115.57) (xy 132.08 120.65))
+  (wire (pts (xy 132.08 109.22) (xy 132.08 110.49))
+    (stroke (width 0) (type default) (color 0 0 0 0))
+  )
+  (wire (pts (xy 139.7 97.79) (xy 139.7 100.33))
+    (stroke (width 0) (type default) (color 0 0 0 0))
+  )
+  (wire (pts (xy 106.68 97.79) (xy 111.76 97.79))
     (stroke (width 0) (type default) (color 0 0 0 0))
   )
@@
     (stroke (width 0) (type default) (color 0 0 0 0))
   )
-  (wire (pts (xy 132.08 102.87) (xy 137.16 102.87))
+  (wire (pts (xy 132.08 109.22) (xy 139.7 109.22))
     (stroke (width 0) (type default) (color 0 0 0 0))
   )
-  (wire (pts (xy 132.08 102.87) (xy 132.08 107.95))
+  (wire (pts (xy 132.08 80.01) (xy 132.08 82.55))
     (stroke (width 0) (type default) (color 0 0 0 0))
   )
-  (wire (pts (xy 132.08 92.71) (xy 132.08 97.79))
+  (wire (pts (xy 139.7 97.79) (xy 142.24 97.79))
+    (stroke (width 0) (type default) (color 0 0 0 0))
+  )
+  (wire (pts (xy 139.7 107.95) (xy 139.7 109.22))
+    (stroke (width 0) (type default) (color 0 0 0 0))
+  )
+  (wire (pts (xy 132.08 90.17) (xy 132.08 97.79))
     (stroke (width 0) (type default) (color 0 0 0 0))
   )
@@
     (effects (font (size 1.27 1.27)) (justify right))
   )
-  (hierarchical_label "Signal_3V3" (shape output) (at 137.16 102.87 0)
+  (hierarchical_label "Signal_3V3" (shape output) (at 142.24 97.79 0)
     (effects (font (size 1.27 1.27)) (justify left))
   )
-  (symbol (lib_id "power:+3V3") (at 132.08 92.71 0) (unit 1)
+  (symbol (lib_id "power:+3V3") (at 132.08 80.01 0) (unit 1)
     (in_bom yes) (on_board yes) (fields_autoplaced)
-    (property "Reference" "#PWR?" (id 0) (at 132.08 96.52 0)
+    (property "Reference" "#PWR?" (id 0) (at 132.08 83.82 0)
       (effects (font (size 1.27 1.27)) hide)
     )
-    (property "Value" "+3V3" (id 1) (at 132.08 87.63 0))
-    (property "Footprint" "" (id 2) (at 132.08 92.71 0)
+    (property "Value" "+3V3" (id 1) (at 132.08 74.93 0))
+    (property "Footprint" "" (id 2) (at 132.08 80.01 0)
       (effects (font (size 1.27 1.27)) hide)
     )
-    (property "Datasheet" "" (id 3) (at 132.08 92.71 0)
+    (property "Datasheet" "" (id 3) (at 132.08 80.01 0)
       (effects (font (size 1.27 1.27)) hide)
     )
@@
       (effects (font (size 1.27 1.27)) (justify left))
     )
-    (property "Value" "600R" (id 1) (at 109.22 90.1699 0)
+    (property "Value" "1k" (id 1) (at 109.22 90.1699 0)
       (effects (font (size 1.27 1.27)) (justify left))
     )
@@
     )
     (property "Datasheet" "~" (id 3) (at 106.68 88.9 0)
+      (effects (font (size 1.27 1.27)) hide)
+    )
+    (pin "1")
+    (pin "2")
+  )
+  (symbol (lib_id "Device:C") (at 139.7 104.14 0) (unit 1)
+    (in_bom yes) (on_board yes) (fields_autoplaced)
+    (property "Reference" "C?" (id 0) (at 143.51 102.8699 0)
+      (effects (font (size 1.27 1.27)) (justify left))
+    )
+    (property "Value" "220nF" (id 1) (at 143.51 105.4099 0)
+      (effects (font (size 1.27 1.27)) (justify left))
+    )
+    (property "Footprint" "" (id 2) (at 140.6652 107.95 0)
+      (effects (font (size 1.27 1.27)) hide)
+    )
+    (property "Datasheet" "~" (id 3) (at 139.7 104.14 0)
       (effects (font (size 1.27 1.27)) hide)
     )
@@
     (pin "4")
   )
-  (symbol (lib_id "Device:R") (at 132.08 111.76 0) (unit 1)
+  (symbol (lib_id "Device:R") (at 132.08 86.36 0) (unit 1)
     (in_bom yes) (on_board yes) (fields_autoplaced)
-    (property "Reference" "R?" (id 0) (at 134.62 110.4899 0)
+    (property "Reference" "R?" (id 0) (at 134.62 85.0899 0)
       (effects (font (size 1.27 1.27)) (justify left))
     )
-    (property "Value" "4k7" (id 1) (at 134.62 113.0299 0)
+    (property "Value" "4k7" (id 1) (at 134.62 87.6299 0)
       (effects (font (size 1.27 1.27)) (justify left))
     )
-    (property "Footprint" "" (id 2) (at 130.302 111.76 90)
+    (property "Footprint" "" (id 2) (at 130.302 86.36 90)
       (effects (font (size 1.27 1.27)) hide)
     )
-    (property "Datasheet" "~" (id 3) (at 132.08 111.76 0)
+    (property "Datasheet" "~" (id 3) (at 132.08 86.36 0)
       (effects (font (size 1.27 1.27)) hide)
     )
@@
     (pin "1")
   )
-  (symbol (lib_id "power:GND") (at 132.08 120.65 0) (unit 1)
+  (symbol (lib_id "power:GND") (at 132.08 110.49 0) (unit 1)
     (in_bom yes) (on_board yes)
-    (property "Reference" "#PWR?" (id 0) (at 132.08 127 0)
+    (property "Reference" "#PWR?" (id 0) (at 132.08 116.84 0)
       (effects (font (size 1.27 1.27)) hide)
     )
-    (property "Value" "GND" (id 1) (at 132.08 125.73 0))
-    (property "Footprint" "" (id 2) (at 132.08 120.65 0)
+    (property "Value" "GND" (id 1) (at 132.08 115.57 0))
+    (property "Footprint" "" (id 2) (at 132.08 110.49 0)
       (effects (font (size 1.27 1.27)) hide)
     )
-    (property "Datasheet" "" (id 3) (at 132.08 120.65 0)
+    (property "Datasheet" "" (id 3) (at 132.08 110.49 0)
       (effects (font (size 1.27 1.27)) hide)
     )
